File: docs/JustBetweenUs.kicad_sch (KiCad schematic)
At the start: 17 parts, among them J1 Eurorack_Power_16pin_Shrouded, J2 USB_B_Micro, J3 USB_B_Micro, J4 Conn_01x05, J8 AudioJack, J9 AudioJack, Q1 BC547, Q2 BC547, SW1 SW_Push, SW2 RotaryEncoder_Switch, U1 Teensy4.1

Commit message: update schematics
Parts:
- removed J1: Eurorack_Power_16pin_Shrouded, 4ms_Connector:Pins_2x08_2.54mm_TH_EuroPower_Shrouded, symbol PCM_4ms_Connector:Eurorack_Power_16pin_Shrouded
- removed J2, J3: USB_B_Micro, symbol Connector:USB_B_Micro
- removed J4: Conn_01x05, symbol Connector_Generic:Conn_01x05
- removed J8, J9: AudioJack, symbol Connector_Audio:AudioJack2_Ground
- removed Q1, Q2: BC547, Package_TO_SOT_THT:TO-92_Inline, symbol Transistor_BJT:BC547
- removed R1, R2, R3, R6: 10k_0603, 4ms_Resistor:R_0603, symbol PCM_4ms_Resistor:10k_0603
- removed R4, R5: 4.7k_0603, 4ms_Resistor:R_0603, symbol PCM_4ms_Resistor:4.7k_0603
- removed SW1: SW_Push, symbol Switch:SW_Push
- removed SW2: RotaryEncoder_Switch, symbol Device:RotaryEncoder_Switch
- removed U1: Teensy4.1, symbol Teensy:Teensy4.1
- added C1 (x2), C2 (x2), C3: 22uF_0805_25V, 4ms_Capacitor:C_0805, symbol PCM_4ms_Capacitor:22uF_0805_25V
- added C10, C11, C12, C13, C14, C4, C5, C6, C9: 100nF_0603_16V, 4ms_Capacitor:C_0603, symbol PCM_4ms_Capacitor:100nF_0603_16V
- added C4, C5: 10uF_0805_25V, 4ms_Capacitor:C_0805, symbol PCM_4ms_Capacitor:10uF_0805_25V
- added J10, J11, J12, J13: AudioJack, symbol Connector_Audio:AudioJack2_Ground
- added J5: PwrHeader, 4ms_Connector:Pins_2x05_2.54mm_TH_Europower, symbol PCM_4ms_Connector:Eurorack_Power_10pin_Unshrouded
- added J6: EurorackPwr, 4ms_Connector:Pins_2x08_2.54mm_TH_EuroPower_Shrouded, symbol PCM_4ms_Connector:Eurorack_Power_16pin_Shrouded
- added KY-1: ~, symbol JBU_Library:KY-040
- added R13, R14, R15, R16, R17, R18, R19, R7: 10k_0603, 4ms_Resistor:R_0603, symbol PCM_4ms_Resistor:10k_0603
- added R20, R9: 4.7k_0603, 4ms_Resistor:R_0603, symbol PCM_4ms_Resistor:4.7k_0603
- added R21, R8: 1k_0603, 4ms_Resistor:R_0603, symbol PCM_4ms_Resistor:1k_0603
- added SW3: SW_Push, symbol Switch:SW_Push
- added Teensy 4.1: ~, symbol JBU_Library:JBU_Teensy
- added U3: LM1117T-5.0, Package_TO_SOT_THT:TO-220-3_Vertical, symbol Regulator_Linear:LM1117T-5.0
- added U4: TL074, symbol Amplifier_Operational:TL074
Connections:
- net +5V: now also C3.1, C5.1, C6.1, J6.5 (+12V), KY-1.2 (+), Teensy 4.1.5v (VIN), U3.2 (VO)
- net GND: now also C11.2, C12.2, C14.2, C4.2, C4.2, C5.1, C5.2, C6.2, C9.2, J10.G, J11.G, J12.G, J13.G, J5.3 (GND), J5.5 (GND), J5.7 (GND), KY-1.1 (GND), R19.2, R7.2, SW3.1, Teensy 4.1.GND, U3.1 (GND)
- new net: R7.1, R9.1, U4.6 (-)
- new net: C3.2, J6.11 (GND)
- new net: C1.2, C2.1, J6.12 (GND)
- new net: C2.2, J6.16 (P16)
- new net: C1.1, J6.8 (+12V)
- new net: R19.1, R20.1, U4.13 (-)
- new net: C13.2, U4.12 (+), U4.8, U4.9 (-)
- new net: R20.2, R21.1, U4.14
- new net: C1.2, C2.1, J5.4 (GND), J5.6 (GND), J5.8 (GND)
- new net: C2.2, J5.10 (-12V), J5.9 (-12V)
- new net: C9.1, R13.1, R14.2
- new net: C11.1, R15.1, U4.3 (+)
- new net: C10.1, R14.1, R15.2
- new net: C5.2, U4.11 (V-)
- new net: J13.T, R21.2
- new net: C1.1, J5.1 (+12V), J5.2 (+12V)
- new net: C4.1, U3.3 (VI)
- new net: C13.1, R17.1, R18.2
- new net: C10.2, U4.1, U4.2 (-), U4.5 (+)
- new net: C12.1, R16.1, R17.2
- new net: C4.1, U4.4 (V+)
- new net: R8.1, R9.2, U4.7
- new net: J12.T, R8.2
- new net: C14.1, R18.1, U4.10 (+)
- new net ENCODER_A: KY-1.5 (CLK), Teensy 4.1.32
- new net ENCODER_B: KY-1.4 (DT), Teensy 4.1.31
- new net ENCODER_SW: KY-1.3 (SW), Teensy 4.1.30
- new net OUTPUT_1: R13.2, Teensy 4.1.24
- new net OUTPUT_2: R16.2, Teensy 4.1.25
- new net Output 1/OUTPUT: J10.T
- new net Output 2/OUTPUT: J11.T
- new net PLAY_BTN: SW3.2, Teensy 4.1.7
Other:
- added sheet Output 1 (output.kicad_sch)
- added sheet Output 2 (output.kicad_sch)
- added sheet old (old.kicad_sch)
- note removed: "Built-in USB connector"
- note removed: "External USB connector VBUS is NOT connected"
- note removed: "KY-040"
- note removed: "Output 1"
- note removed: "Output 2"

Commit message: powerLayout
updated power layout with a sub page in the root schematic
Parts:
- removed C1 (x2), C2 (x2), C3: 22uF_0805_25V, 4ms_Capacitor:C_0805, symbol PCM_4ms_Capacitor:22uF_0805_25V
- removed C10, C11, C12, C13, C14, C4, C5, C6, C9: 100nF_0603_16V, 4ms_Capacitor:C_0603, symbol PCM_4ms_Capacitor:100nF_0603_16V
- removed C4, C5: 10uF_0805_25V, 4ms_Capacitor:C_0805, symbol PCM_4ms_Capacitor:10uF_0805_25V
- removed J10, J11, J12, J13: AudioJack, symbol Connector_Audio:AudioJack2_Ground
- removed J5: PwrHeader, 4ms_Connector:Pins_2x05_2.54mm_TH_Europower, symbol PCM_4ms_Connector:Eurorack_Power_10pin_Unshrouded
- removed J6: EurorackPwr, 4ms_Connector:Pins_2x08_2.54mm_TH_EuroPower_Shrouded, symbol PCM_4ms_Connector:Eurorack_Power_16pin_Shrouded
- removed KY-1: ~, symbol JBU_Library:KY-040
- removed R13, R14, R15, R16, R17, R18, R19, R7: 10k_0603, 4ms_Resistor:R_0603, symbol PCM_4ms_Resistor:10k_0603
- removed R20, R9: 4.7k_0603, 4ms_Resistor:R_0603, symbol PCM_4ms_Resistor:4.7k_0603
- removed R21, R8: 1k_0603, 4ms_Resistor:R_0603, symbol PCM_4ms_Resistor:1k_0603
- removed SW3: SW_Push, symbol Switch:SW_Push
- removed Teensy 4.1: ~, symbol JBU_Library:JBU_Teensy
- removed U3: LM1117T-5.0, Package_TO_SOT_THT:TO-220-3_Vertical, symbol Regulator_Linear:LM1117T-5.0
- removed U4: TL074, symbol Amplifier_Operational:TL074
- added J2, J3: USB_B_Micro, symbol Connector:USB_B_Micro
- added J4: Conn_01x05, symbol Connector_Generic:Conn_01x05
- added J8, J9: AudioJack, symbol Connector_Audio:AudioJack2_Ground
- added Q1, Q2: BC547, Package_TO_SOT_THT:TO-92_Inline, symbol Transistor_BJT:BC547
- added R1, R2, R3, R6: 10k_0603, 4ms_Resistor:R_0603, symbol PCM_4ms_Resistor:10k_0603
- added R4, R5: 4.7k_0603, 4ms_Resistor:R_0603, symbol PCM_4ms_Resistor:4.7k_0603
- added SW1: SW_Push, symbol Switch:SW_Push
- added SW2: RotaryEncoder_Switch, symbol Device:RotaryEncoder_Switch
- added U1: Teensy4.1, symbol Teensy:Teensy4.1
Connections:
- net +5V: now also J4.+, R1.2, R2.1, R4.1, R5.1, U1.48 (VIN)
- net GND: now also J2.5 (GND), J2.6 (Shield), J3.5 (GND), J3.6 (Shield), J4.GND, J8.G, J9.G, Q1.3 (E), Q2.3 (E), SW1.1, SW2.C, SW2.S2, U1.47 (GND)
- new net: J4.CLK, R1.1, SW2.A, U1.24 (32_OUT1B)
- new net: J2.1 (VBUS), U1.49 (VUSB)
- new net: J2.2 (D-), J3.2 (D-), U1.66 (D-)
- new net: J2.3 (D+), J3.3 (D+), U1.67 (D+)
- new net: J4.DT, R2.2, SW2.B, U1.23 (31_CTX3)
- new net: J4.SW, SW2.S1, U1.22 (30_CRX3)
- new net: Q1.2 (B), R3.1
- new net: R3.2, U1.16 (24_A10_TX6_SCL2)
- new net: SW1.2, U1.9 (7_RX2_OUT1A)
- new net: J8.T, Q2.1 (C), R5.2
- new net: Q2.2 (B), R6.1
- new net: J9.T, Q1.1 (C), R4.2
- new net: R6.2, U1.17 (25_A11_RX6_SDA2)
Other:
- removed sheet Output 1
- removed sheet Output 2
- removed sheet old
- added sheet power (power.kicad_sch)
- note added: "Built-in USB connector"
- note added: "External USB connector VBUS is NOT connected"
- note added: "KY-040"
- note added: "Output 1"
- note added: "Output 2"
